File: boards/parallella-porcupine/porcu-elink-north.sch (KiCad schematic (older format))
At the start: 4 parts, among them J15 CONN\\HDR\\P1\\2R15\\SHD, J16 CONN\\HDR\\P1\\2R15\\SHD, J17 CONN\\HDR\\P1\\1R15, J18 CONN\\HDR\\P1\\1R15

Commit message: Schematic is stable, PCB mostly routed.
Parts:
- removed J15, J16: CONN\\HDR\\P1\\2R15\\SHD, CONN_HDR_P1_2R15_SHD, symbol CONN\HDR\P1\2R15\SHD
- removed J17, J18: CONN\\HDR\\P1\\1R15, CONN_HDR_P1_1R15, symbol CONN\HDR\P1\1R15
- added J17, J18: CONN\\HDR\\2MM\\2R15\\SHD, CONN_HDR_2MM_2R15_SHD, symbol CONN\HDR\2MM\2R15\SHD
- added J19, J20: CONN\\HDR\\2MM\\1R15, CONN_HDR_2MM_1R15, symbol CONN\HDR\2MM\1R15
Other:
- note added: "NOTE: Single-row headers are to be \nplaced 2mm from "even" side of dual-row \nheaders. In this way the polarity of all \nsignals may be reversed to support \nE64 chips by shifting the dual-row \ncomponent such that it uses the \n"even" side of the dual-row footprint \nplus the single-row footprint.\n"
- note removed: "NOTE: Single-row headers are to be \nplaced 0.1" from "even" side of dual-row \nheaders. In this way the polarity of all \nsignals may be reversed to support \nE64 chips by shifting the dual-row \ncomponent such that it uses the \n"even" side of the dual-row footprint \nplus the single-row footprint.\n"
Changed lines of the file:
@@
 TXO_DATA_N[0..7]
 $Comp
-L GND #PWR025
+L GND #PWR029
 U 1 1 538F4EDB
 P 5250 5750
-F 0 "#PWR025" H 5250 5750 30  0001 C CNN
+F 0 "#PWR029" H 5250 5750 30  0001 C CNN
 F 1 "GND" H 5250 5680 30  0001 C CNN
 F 2 "" H 5250 5750 60  0000 C CNN
@@
 $EndComp
 $Comp
-L GND #PWR026
+L GND #PWR030
 U 1 1 538F4EDC
 P 4450 5750
-F 0 "#PWR026" H 4450 5750 30  0001 C CNN
+F 0 "#PWR030" H 4450 5750 30  0001 C CNN
 F 1 "GND" H 4450 5680 30  0001 C CNN
 F 2 "" H 4450 5750 60  0000 C CNN
@@
 	3550 2500 3650 2600
 $Comp
-L GND #PWR027
+L GND #PWR031
 U 1 1 538EA4B2
 P 5250 3250
-F 0 "#PWR027" H 5250 3250 30  0001 C CNN
+F 0 "#PWR031" H 5250 3250 30  0001 C CNN
 F 1 "GND" H 5250 3180 30  0001 C CNN
 F 2 "" H 5250 3250 60  0000 C CNN
@@
 $EndComp
 $Comp
-L GND #PWR028
+L GND #PWR032
 U 1 1 538EA4C6
 P 4450 3250
-F 0 "#PWR028" H 4450 3250 30  0001 C CNN
+F 0 "#PWR032" H 4450 3250 30  0001 C CNN
 F 1 "GND" H 4450 3180 30  0001 C CNN
 F 2 "" H 4450 3250 60  0000 C CNN
@@
 RXI_FRAME_P
 $Comp
-L GND #PWR029
+L GND #PWR033
 U 1 1 538F441C
 P 7500 3400
-F 0 "#PWR029" H 7500 3400 30  0001 C CNN
+F 0 "#PWR033" H 7500 3400 30  0001 C CNN
 F 1 "GND" H 7500 3330 30  0001 C CNN
 F 2 "" H 7500 3400 60  0000 C CNN
@@
 RXI_DATA_P[0..7]
 Text Notes 8700 2400 0    60   ~ 0
-NOTE:  Single-row headers are to be \nplaced 0.1" from "even" side of dual-row \nheaders.  In this way the polarity of all \nsignals may be reversed to support \nE64 chips by shifting the dual-row \ncomponent such that it uses the \n"even" side of the dual-row footprint \nplus the single-row footprint.\n
+NOTE:  Single-row headers are to be \nplaced 2mm from "even" side of dual-row \nheaders.  In this way the polarity of all \nsignals may be reversed to support \nE64 chips by shifting the dual-row \ncomponent such that it uses the \n"even" side of the dual-row footprint \nplus the single-row footprint.\n
 Text Label 7600 4950 0    60   ~ 0
 TXO_DATA_P1
@@
 TXO_FRAME_P
 $Comp
-L GND #PWR030
+L GND #PWR034
 U 1 1 538F45E6
 P 7500 5850
-F 0 "#PWR030" H 7500 5850 30  0001 C CNN
+F 0 "#PWR034" H 7500 5850 30  0001 C CNN
 F 1 "GND" H 7500 5780 30  0001 C CNN
 F 2 "" H 7500 5850 60  0000 C CNN
@@
 TXO_DATA_P[0..7]
 $Comp
-L CONN\HDR\P1\2R15\SHD J15
-U 1 1 538F80D6
+L CONN\HDR\2MM\2R15\SHD J17
+U 1 1 53976F8A
 P 4850 2400
-F 0 "J15" H 4500 3250 60  0000 C CNN
-F 1 "CONN\\HDR\\P1\\2R15\\SHD" H 4850 3550 60  0001 C CNN
-F 2 "CONN_HDR_P1_2R15_SHD" H 4850 3350 60  0000 C CNN
+F 0 "J17" H 4500 3250 60  0000 C CNN
+F 1 "CONN\\HDR\\2MM\\2R15\\SHD" H 4850 3550 60  0001 C CNN
+F 2 "CONN_HDR_2MM_2R15_SHD" H 4850 3350 60  0000 C CNN
 F 3 "" H 4850 3300 60  0001 C CNN
-F 4 "302-S301" H 4850 3250 50  0000 C CNN "MFRPN"
-F 5 "On-Shore_Tech." H 4850 3450 50  0001 C CNN "MFR"
+F 4 "0878313020" H 4875 3250 50  0000 C CNN "MFRPN"
+F 5 "Molex" H 4850 3450 50  0001 C CNN "MFR"
 	1    4850 2400
 	1    0    0    -1
 $EndComp
 $Comp
-L CONN\HDR\P1\2R15\SHD J16
-U 1 1 538F80F8
+L CONN\HDR\2MM\2R15\SHD J18
+U 1 1 53976FAC
 P 4850 4850
-F 0 "J16" H 4500 5700 60  0000 C CNN
-F 1 "CONN\\HDR\\P1\\2R15\\SHD" H 4850 6000 60  0001 C CNN
-F 2 "CONN_HDR_P1_2R15_SHD" H 4850 5800 60  0000 C CNN
+F 0 "J18" H 4500 5700 60  0000 C CNN
+F 1 "CONN\\HDR\\2MM\\2R15\\SHD" H 4850 6000 60  0001 C CNN
+F 2 "CONN_HDR_2MM_2R15_SHD" H 4850 5800 60  0000 C CNN
 F 3 "" H 4850 5750 60  0001 C CNN
-F 4 "302-S301" H 4850 5700 50  0000 C CNN "MFRPN"
-F 5 "On-Shore_Tech." H 4850 5900 50  0001 C CNN "MFR"
+F 4 "0878313020" H 4875 5700 50  0000 C CNN "MFRPN"
+F 5 "Molex" H 4850 5900 50  0001 C CNN "MFR"
 	1    4850 4850
 	1    0    0    -1
 $EndComp
 $Comp
-L CONN\HDR\P1\1R15 J18
-U 1 1 538F811A
+L CONN\HDR\2MM\1R15 J19
+U 1 1 53976FCE
+P 7150 2400
+F 0 "J19" H 6850 3250 60  0000 C CNN
+F 1 "CONN\\HDR\\2MM\\1R15" H 7200 3550 60  0001 C CNN
+F 2 "CONN_HDR_2MM_1R15" V 7300 2400 60  0000 C CNN
+F 3 "" H 7200 3300 60  0001 C CNN
+F 4 "951115-8622-AR" H 7350 3250 50  0001 C CNN "MFRPN"
+F 5 "3M" H 7200 3450 50  0001 C CNN "MFR"
+F 6 "DNI" H 6550 3250 60  0000 C CNN "DNI"
+	1    7150 2400
+	-1   0    0    -1
+$EndComp
+$Comp
+L CONN\HDR\2MM\1R15 J20
+U 1 1 53976FF0
 P 7150 4850
-F 0 "J18" H 6850 5700 60  0000 C CNN
-F 1 "CONN\\HDR\\P1\\1R15" H 7200 6000 60  0001 C CNN
-F 2 "CONN_HDR_P1_1R15" H 7200 5800 60  0001 C CNN
+F 0 "J20" H 6850 5700 60  0000 C CNN
+F 1 "CONN\\HDR\\2MM\\1R15" H 7200 6000 60  0001 C CNN
+F 2 "CONN_HDR_2MM_1R15" V 7300 4850 60  0000 C CNN
 F 3 "" H 7200 5750 60  0001 C CNN
-F 4 "PRPC015SAAN-RC" H 7350 5700 50  0001 C CNN "MFRPN"
-F 5 "Sullins" H 7200 5900 50  0001 C CNN "MFR"
-F 6 "DNI" H 7100 5700 60  0000 C CNN "DNI"
+F 4 "951115-8622-AR" H 7350 5700 50  0001 C CNN "MFRPN"
+F 5 "3M" H 7200 5900 50  0001 C CNN "MFR"
+F 6 "DNI" H 6600 5700 60  0000 C CNN "DNI"
 	1    7150 4850
 	-1   0    0    -1
 $EndComp
-$Comp
-L CONN\HDR\P1\1R15 J17
-U 1 1 538F813C
-P 7150 2400
-F 0 "J17" H 6850 3250 60  0000 C CNN
-F 1 "CONN\\HDR\\P1\\1R15" H 7200 3550 60  0001 C CNN
-F 2 "CONN_HDR_P1_1R15" H 7200 3350 60  0001 C CNN
-F 3 "" H 7200 3300 60  0001 C CNN
-F 4 "PRPC015SAAN-RC" H 7350 3250 50  0001 C CNN "MFRPN"
-F 5 "Sullins" H 7200 3450 50  0001 C CNN "MFR"
-F 6 "DNI" H 7100 3250 60  0000 C CNN "DNI"
-	1    7150 2400
-	-1   0    0    -1
-$EndComp
