File: boards/parallella-porcupine/porcu-elink-south.sch (KiCad schematic (older format))
At the start: 2 parts, among them J19 CONN\\HDR\\P1\\2R15\\SHD, J20 CONN\\HDR\\P1\\2R15\\SHD

Commit message: Schematic is stable, PCB mostly routed.
Parts:
- removed J19, J20: CONN\\HDR\\P1\\2R15\\SHD, CONN_HDR_P1_2R15_SHD, symbol CONN\HDR\P1\2R15\SHD
- added J21, J22: CONN\\HDR\\2MM\\2R15\\SHD, CONN_HDR_2MM_2R15_SHD, symbol CONN\HDR\2MM\2R15\SHD
Changed lines of the file:
@@
 Rev "*"
 Comp "Adapteva, Inc., 1666 Massachusetts Ave., Lexington, MA, 02420"
-Comment1 "Elink Connectors"
+Comment1 "Elink South Connectors"
 Comment2 ""
 Comment3 ""
@@
 TXO_DATA_N[0..7]
 $Comp
-L GND #PWR033
+L GND #PWR037
 U 1 1 538E831F
 P 5250 5750
-F 0 "#PWR033" H 5250 5750 30  0001 C CNN
+F 0 "#PWR037" H 5250 5750 30  0001 C CNN
 F 1 "GND" H 5250 5680 30  0001 C CNN
 F 2 "" H 5250 5750 60  0000 C CNN
@@
 $EndComp
 $Comp
-L GND #PWR034
+L GND #PWR038
 U 1 1 538E9F0A
 P 4450 5750
-F 0 "#PWR034" H 4450 5750 30  0001 C CNN
+F 0 "#PWR038" H 4450 5750 30  0001 C CNN
 F 1 "GND" H 4450 5680 30  0001 C CNN
 F 2 "" H 4450 5750 60  0000 C CNN
@@
 	3550 2500 3650 2600
 $Comp
-L GND #PWR035
+L GND #PWR039
 U 1 1 538F4EDD
 P 5250 3250
-F 0 "#PWR035" H 5250 3250 30  0001 C CNN
+F 0 "#PWR039" H 5250 3250 30  0001 C CNN
 F 1 "GND" H 5250 3180 30  0001 C CNN
 F 2 "" H 5250 3250 60  0000 C CNN
@@
 $EndComp
 $Comp
-L GND #PWR036
+L GND #PWR040
 U 1 1 538F4EDE
 P 4450 3250
-F 0 "#PWR036" H 4450 3250 30  0001 C CNN
+F 0 "#PWR040" H 4450 3250 30  0001 C CNN
 F 1 "GND" H 4450 3180 30  0001 C CNN
 F 2 "" H 4450 3250 60  0000 C CNN
@@
 Connection ~ 5250 2800
 $Comp
-L CONN\HDR\P1\2R15\SHD J19
-U 1 1 538F8815
+L CONN\HDR\2MM\2R15\SHD J21
+U 1 1 53977A3A
 P 4850 2400
-F 0 "J19" H 4500 3250 60  0000 C CNN
-F 1 "CONN\\HDR\\P1\\2R15\\SHD" H 4850 3550 60  0001 C CNN
-F 2 "CONN_HDR_P1_2R15_SHD" H 4850 3350 60  0000 C CNN
+F 0 "J21" H 4500 3250 60  0000 C CNN
+F 1 "CONN\\HDR\\2MM\\2R15\\SHD" H 4850 3550 60  0001 C CNN
+F 2 "CONN_HDR_2MM_2R15_SHD" H 4850 3350 60  0000 C CNN
 F 3 "" H 4850 3300 60  0001 C CNN
-F 4 "302-S301" H 4850 3250 50  0000 C CNN "MFRPN"
-F 5 "On-Shore_Tech." H 4850 3450 50  0001 C CNN "MFR"
+F 4 "0878313020" H 4875 3250 50  0000 C CNN "MFRPN"
+F 5 "Molex" H 4850 3450 50  0001 C CNN "MFR"
 	1    4850 2400
 	1    0    0    -1
 $EndComp
 $Comp
-L CONN\HDR\P1\2R15\SHD J20
-U 1 1 538F8845
+L CONN\HDR\2MM\2R15\SHD J22
+U 1 1 53977A5C
 P 4850 4850
-F 0 "J20" H 4500 5700 60  0000 C CNN
-F 1 "CONN\\HDR\\P1\\2R15\\SHD" H 4850 6000 60  0001 C CNN
-F 2 "CONN_HDR_P1_2R15_SHD" H 4850 5800 60  0000 C CNN
+F 0 "J22" H 4500 5700 60  0000 C CNN
+F 1 "CONN\\HDR\\2MM\\2R15\\SHD" H 4850 6000 60  0001 C CNN
+F 2 "CONN_HDR_2MM_2R15_SHD" H 4850 5800 60  0000 C CNN
 F 3 "" H 4850 5750 60  0001 C CNN
-F 4 "302-S301" H 4850 5700 50  0000 C CNN "MFRPN"
-F 5 "On-Shore_Tech." H 4850 5900 50  0001 C CNN "MFR"
+F 4 "0878313020" H 4875 5700 50  0000 C CNN "MFRPN"
+F 5 "Molex" H 4850 5900 50  0001 C CNN "MFR"
 	1    4850 4850
 	1    0    0    -1
