File: boards/parallella-porcupine/porcupine.kicad_pcb (KiCad board)
At the start: 6 copper layers, 86.4 x 54.6 mm, 35 parts, among them J1 CONN\HDR\P1\2R15, J11 CONN\HDR\2MM\2R07\SHD, J12 CONN\HDR\P1\1R02, J13 CONN\HDR\P1\1R02, J14 CONN\HDR\P1\2R15, J15 CONN\HDR\2MM\2R15\SHD, J16 CONN\HDR\2MM\2R15\SHD, J17 CONN\HDR\2MM\2R15\SHD, J18 CONN\HDR\2MM\2R15\SHD, J3 CONN\HDR\P1FRA\2R06, J4 CONN\HDR\P1\2R15, J5 CONN\HDR\P1\2R15, P1 CONN\SAMTEC\BTH\60, P2 CONN\SAMTEC\BTH\60, P3 CONN\SAMTEC\BTH\60, P4 CONN\SAMTEC\BTH\60

Commit message: Ready for full review.
Parts:
- removed J12: CONN\HDR\P1\1R02, Adapteva:CONN_HDR_P1_1R02
- removed R9: 1k00, R_0805_HS
- added G***: LOGO, Adapteva:adapteva_logo, F.Cu at (174.0, 108.0)
- moved FID3 8.89 mm to (155.6, 123.8)
- moved FID4 8.89 mm to (155.6, 123.8)
- moved J10 8.89 mm to (206.4, 142.9)
- moved J11 8.89 mm to (206.4, 134.0)
- renumbered FID4 to FID2, FID2 to FID3, FID5 to FID4, FID3 to FID5, J11 to J1, J17 to J10, J18 to J11, J1 to J2, J14 to J3, J13 to J4, J3 to J5, J4 to J6, J5 to J7, J15 to J8, J16 to J9, P3 to P1, P1 to P2, P2 to P3
Connections:
- J2 pad 10: /POWER/UART_TX -> /POWER/PROG_IO
- J2 pad 11: /POWER/PROG_IO -> /POWER/UART_TX
- J2 pad 12: /POWER/UART_RX -> /POWER/I2C_SDA
- J2 pad 13: /POWER/VDD_ADJ -> /POWER/UART_RX
- J2 pad 14: /POWER/VDD_GPIO -> /POWER/I2C_SCL
- J2 pad 15: /POWER/1P8V -> GND
- J2 pad 16: /POWER/1P8V -> GND
- J2 pad 17: /POWER/DSP_XID3 -> /POWER/3P3V
- J2 pad 18: /POWER/DSP_YID3 -> /POWER/SYS_5P0V
- J2 pad 19: /POWER/DSP_XID2 -> /POWER/VDD_ADJ
- J2 pad 20: /POWER/DSP_YID2 -> /POWER/VDD_GPIO
- J2 pad 21: /POWER/DSP_XID1 -> /POWER/1P8V
- J2 pad 22: /POWER/DSP_YID1 -> /POWER/JTAG_BOOT_EN
- J2 pad 23: /POWER/DSP_XID0 -> /POWER/DSP_XID3
- J2 pad 24: /POWER/DSP_YID0 -> /POWER/DSP_YID3
- J2 pad 25: GND -> /POWER/DSP_XID2
- J2 pad 26: GND -> /POWER/DSP_YID2
- J2 pad 27: /POWER/I2C_SCL -> /POWER/DSP_XID1
- J2 pad 28: /POWER/I2C_SDA -> /POWER/DSP_YID1
- J2 pad 29: /POWER/SYS_5P0V -> /POWER/DSP_XID0
- J2 pad 30: /POWER/3P3V -> /POWER/DSP_YID0
- J3 pad 17: (no net) -> /POWER/SPARE
- P1 pad 10: (no net) -> /POWER/SPARE
Routing:
- net /POWER/I2C_SDA: track 30.6 -> 55.5 mm
- net /POWER/I2C_SCL: track 26.2 -> 50.5 mm
- net /P_ELINK_S/RXI_DATA_N0: track 32.3 -> 8.56 mm, vias 1 -> 0
- net /P_ELINK_S/RXI_DATA_P0: track 28.9 -> 5.94 mm, vias 1 -> 0
- net /P_ELINK_S/TXO_DATA_P4: track 8.27 -> 26.3 mm, vias 0 -> 1
- net /P_ELINK_S/RXI_DATA_N6: track 34.9 -> 17.2 mm, vias 1 -> 0
- net /P_ELINK_S/RXI_DATA_N1: track 30.8 -> 14.4 mm
- net /P_ELINK_S/RXI_DATA_P6: track 30.9 -> 15.4 mm, vias 1 -> 0
- net /P_ELINK_S/TXO_DATA_N4: track 10.9 -> 26.2 mm, vias 0 -> 1
- net /P_ELINK_S/TXO_DATA_N6: track 8.39 -> 22.5 mm, vias 0 -> 1
- net /P_ELINK_S/TXO_DATA_P6: track 6.19 -> 19.7 mm, vias 0 -> 1
- net /P_ELINK_S/RXI_DATA_P1: track 25.6 -> 12.2 mm
- net /P_ELINK_S/TXO_DATA_P2: track 10.5 -> 23.9 mm, vias 0 -> 1
- net /P_ELINK_S/RXI_DATA_N2: track 21.7 -> 9.96 mm, vias 1 -> 0
- net /P_ELINK_S/RXI_DATA_N7: track 37.5 -> 25.9 mm
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- added copper zone on F.Cu, net /POWER/VDD_ADJ
- added copper zone on B.Cu, net /POWER/VDD_GPIO
- removed copper zone on Inner2.Cu, net /POWER/VDD_ADJ
- removed copper zone on Inner1.Cu, net /POWER/VDD_GPIO
Other:
- board text added: "1 0 RW G"
- board text added: "3 2 1 0 -XID"
- board text added: "3 2 1 0 -YID"
- board text added: "4 3 2 G"
- board text added: "7 6 5 G"
- board text added: "AN G SP"
- board text added: "AP G RN"
- board text added: "G 33 VA 18"
- board text added: "G 50 VG JB"
- board text added: "LC WW FR"
- board text added: "P N"
- board text added: "PN"
- board text added: "TM DF TX RX"
- board text added: "UL PI SD SC"
- board text removed: "ADAPTEVA, INC."
- board text removed: "X3 2 1 0"
- board text removed: "Y3 2 1 0"
