File: boards/parallella-porcupine/paracard-gpio.sch (KiCad schematic (older format))
At the start: 1 part, among them P1 CONN\\SAMTEC\\BTH\\60

Commit message: Completed design w/3-row XID/YID and various 4-pin IO connectors. Fixed page ordering, changed "Mfr" field to "Manufacturer" Will now re-do to combine all misc. functions onto a single 2xN connector.
Parts:
- P1: MFR Samtec -> (none); Manufacturer (none) -> Samtec
Changed lines of the file:
@@
 $Descr B 17000 11000
 encoding utf-8
-Sheet 2 10
+Sheet 3 10
 Title "Parallella Breakout Daughtercard"
 Date "09 May 2014"
@@
 	9200 3900 9300 4000
 $Comp
-L GND #PWR01
+L GND #PWR03
 U 1 1 5386382E
 P 8850 6700
-F 0 "#PWR01" H 8850 6700 30  0001 C CNN
+F 0 "#PWR03" H 8850 6700 30  0001 C CNN
 F 1 "GND" H 8850 6630 30  0001 C CNN
 F 2 "" H 8850 6700 60  0000 C CNN
@@
 $EndComp
 $Comp
-L GND #PWR02
+L GND #PWR04
 U 1 1 538638A0
 P 11950 6700
-F 0 "#PWR02" H 11950 6700 30  0001 C CNN
+F 0 "#PWR04" H 11950 6700 30  0001 C CNN
 F 1 "GND" H 11950 6630 30  0001 C CNN
 F 2 "" H 11950 6700 60  0000 C CNN
@@
 F 1 "CONN\\SAMTEC\\BTH\\60" V 10350 5150 60  0000 C CNN
 F 2 "CONN_SAMTEC_BTH_60" V 10550 5150 60  0001 C CNN
-F 3 "/mnt/windowsC/Adapteva/Fred-suppliers/Suppliers/www.samtec.com/BTH-XXX-XX-X-D-XX-MKT.pdf" H 10550 6050 60  0001 C CNN
+F 3 "" H 10550 6050 60  0001 C CNN
 F 4 "BTH-030-01-F-D-A" V 10450 5150 80  0000 C CNN "MFRPN"
-F 5 "Samtec" V 10450 3950 60  0000 C CNN "MFR"
+F 5 "Samtec" V 10450 3950 60  0000 C CNN "Manufacturer"
 	1    10450 5150
 	1    0    0    -1

Commit message: Ready for full review.
Parts:
- renumbered P1 to P2
Changed lines of the file:
@@
 Sheet 3 10
 Title "Parallella Breakout Daughtercard"
-Date "09 May 2014"
+Date "19 Jun 2014"
 Rev "*"
 Comp "Adapteva, Inc., 1666 Massachusetts Ave., Lexington, MA, 02420"
-Comment1 "Porcupin Top Level"
+Comment1 "Parallella GPIO Connector"
 Comment2 ""
 Comment3 ""
@@
 	8650 3000 11750 3000
 $Comp
-L CONN\SAMTEC\BTH\60 P1
+L CONN\SAMTEC\BTH\60 P2
 U 1 1 538932DF
 P 10450 5150
-F 0 "P1" H 10450 6850 60  0000 C CNN
+F 0 "P2" H 10450 6850 60  0000 C CNN
 F 1 "CONN\\SAMTEC\\BTH\\60" V 10350 5150 60  0000 C CNN
 F 2 "CONN_SAMTEC_BTH_60" V 10550 5150 60  0001 C CNN
