File: boards/parallella-porcupine/paracard-power.sch (KiCad schematic (older format))
At the start: 1 part, among them P3 CONN\\SAMTEC\\BTH\\60

Commit message: Completed design w/3-row XID/YID and various 4-pin IO connectors. Fixed page ordering, changed "Mfr" field to "Manufacturer" Will now re-do to combine all misc. functions onto a single 2xN connector.
Parts:
- P3: MFR Samtec -> (none); Manufacturer (none) -> Samtec
Changed lines of the file:
@@
 $Descr B 17000 11000
 encoding utf-8
-Sheet 4 10
+Sheet 2 10
 Title "Parallella Breakout Daughtercard"
 Date "09 May 2014"
@@
 POWER
 $Comp
-L GND #PWR05
+L GND #PWR01
 U 1 1 53864BC9
 P 8450 6850
-F 0 "#PWR05" H 8450 6850 30  0001 C CNN
+F 0 "#PWR01" H 8450 6850 30  0001 C CNN
 F 1 "GND" H 8450 6780 30  0001 C CNN
 F 2 "" H 8450 6850 60  0000 C CNN
@@
 $EndComp
 $Comp
-L GND #PWR06
+L GND #PWR02
 U 1 1 53864BDD
 P 9850 6850
-F 0 "#PWR06" H 9850 6850 30  0001 C CNN
+F 0 "#PWR02" H 9850 6850 30  0001 C CNN
 F 1 "GND" H 9850 6780 30  0001 C CNN
 F 2 "" H 9850 6850 60  0000 C CNN
@@
 F 1 "CONN\\SAMTEC\\BTH\\60" V 9050 5050 60  0000 C CNN
 F 2 "CONN_SAMTEC_BTH_60" V 9250 5050 60  0001 C CNN
-F 3 "/mnt/windowsC/Adapteva/Fred-suppliers/Suppliers/www.samtec.com/BTH-XXX-XX-X-D-XX-MKT.pdf" H 9250 5950 60  0001 C CNN
+F 3 "" H 9250 5950 60  0001 C CNN
 F 4 "BTH-030-01-F-D-A" V 9150 5050 80  0000 C CNN "MFRPN"
-F 5 "Samtec" V 9150 3850 60  0000 C CNN "MFR"
+F 5 "Samtec" V 9150 3850 60  0000 C CNN "Manufacturer"
 	1    9150 5050
 	1    0    0    -1

Commit message: Ready for full review.
Parts:
- renumbered P3 to P1
Connections:
- net labels added: SPARE
- wire segments 64 -> 65
- no-connect marks 1 -> 0
Changed lines of the file:
@@
 Sheet 2 10
 Title "Parallella Breakout Daughtercard"
-Date "09 May 2014"
+Date "19 Jun 2014"
 Rev "*"
 Comp "Adapteva, Inc., 1666 Massachusetts Ave., Lexington, MA, 02420"
-Comment1 "Porcupin Top Level"
+Comment1 "Parallella Power Connector"
 Comment2 ""
 Comment3 ""
@@
 Text HLabel 5850 4650 0    60   Input ~ 0
 REG_EN[1..4]
-NoConn ~ 8650 4000
 Text HLabel 10550 4000 2    60   BiDi ~ 0
 PROG_IO
@@
 	9850 3250 8250 3250
 $Comp
-L CONN\SAMTEC\BTH\60 P3
+L CONN\SAMTEC\BTH\60 P1
 U 1 1 538934D7
 P 9150 5050
-F 0 "P3" H 9150 6750 60  0000 C CNN
+F 0 "P1" H 9150 6750 60  0000 C CNN
 F 1 "CONN\\SAMTEC\\BTH\\60" V 9050 5050 60  0000 C CNN
 F 2 "CONN_SAMTEC_BTH_60" V 9250 5050 60  0001 C CNN
@@
 	1    0    0    -1
 $EndComp
+Text HLabel 7750 4000 0    60   BiDi ~ 0
+SPARE
+Wire Wire Line
+	7750 4000 8650 4000
 $EndSCHEMATC
