File: boards/parallella-porcupine/porcu-elink.sch (KiCad schematic (older format))
At the start: 2 parts, among them J15 CONN\\HDR\\2MM\\2R15\\SHD, J16 CONN\\HDR\\2MM\\2R15\\SHD

Commit message: Completed design w/3-row XID/YID and various 4-pin IO connectors. Fixed page ordering, changed "Mfr" field to "Manufacturer" Will now re-do to combine all misc. functions onto a single 2xN connector.
Parts:
- J15, J16: MFR Molex -> (none); Manufacturer (none) -> Molex
Changed lines of the file:
@@
 TXO_DATA_N[0..7]
 $Comp
-L GND #PWR026
+L GND #PWR028
 U 1 1 538E831F
 P 8850 6950
-AR Path="/538C99D9/538E831F" Ref="#PWR026"  Part="1"
+AR Path="/538C99D9/538E831F" Ref="#PWR028"  Part="1"
 AR Path="/538F26CD/538E831F" Ref="#PWR032"  Part="1"
 F 0 "#PWR032" H 8850 6950 30  0001 C CNN
@@
 $EndComp
 $Comp
-L GND #PWR027
+L GND #PWR029
 U 1 1 538E9F0A
 P 8050 6950
-AR Path="/538C99D9/538E9F0A" Ref="#PWR027"  Part="1"
+AR Path="/538C99D9/538E9F0A" Ref="#PWR029"  Part="1"
 AR Path="/538F26CD/538E9F0A" Ref="#PWR033"  Part="1"
 F 0 "#PWR033" H 8050 6950 30  0001 C CNN
@@
 	7150 3700 7250 3800
 $Comp
-L GND #PWR028
+L GND #PWR030
 U 1 1 538F4EDD
 P 8850 4450
-AR Path="/538C99D9/538F4EDD" Ref="#PWR028"  Part="1"
+AR Path="/538C99D9/538F4EDD" Ref="#PWR030"  Part="1"
 AR Path="/538F26CD/538F4EDD" Ref="#PWR034"  Part="1"
 F 0 "#PWR034" H 8850 4450 30  0001 C CNN
@@
 $EndComp
 $Comp
-L GND #PWR029
+L GND #PWR031
 U 1 1 538F4EDE
 P 8050 4450
-AR Path="/538C99D9/538F4EDE" Ref="#PWR029"  Part="1"
+AR Path="/538C99D9/538F4EDE" Ref="#PWR031"  Part="1"
 AR Path="/538F26CD/538F4EDE" Ref="#PWR035"  Part="1"
 F 0 "#PWR035" H 8050 4450 30  0001 C CNN
@@
 F 3 "" H 8450 4500 60  0001 C CNN
 F 4 "0878313020" H 8475 4450 50  0000 C CNN "MFRPN"
-F 5 "Molex" H 8450 4650 50  0001 C CNN "MFR"
+F 5 "Molex" H 8450 4650 50  0001 C CNN "Manufacturer"
 	1    8450 3600
 	1    0    0    -1
@@
 F 3 "" H 8450 6950 60  0001 C CNN
 F 4 "0878313020" H 8475 6900 50  0000 C CNN "MFRPN"
-F 5 "Molex" H 8450 7100 50  0001 C CNN "MFR"
+F 5 "Molex" H 8450 7100 50  0001 C CNN "Manufacturer"
 	1    8450 6050
 	1    0    0    -1

Commit message: Ready for full review.
Parts:
- renumbered J15 to J8, J16 to J9
Changed lines of the file:
@@
 $Descr B 17000 11000
 encoding utf-8
-Sheet 10 10
+Sheet 9 10
 Title "Parallella Breakout Daughtercard"
-Date "09 May 2014"
+Date "19 Jun 2014"
 Rev "*"
 Comp "Adapteva, Inc., 1666 Massachusetts Ave., Lexington, MA, 02420"
@@
 TXO_DATA_N[0..7]
 $Comp
-L GND #PWR024
+L GND #PWR023
 U 1 1 538E831F
 P 8850 6950
-AR Path="/538C99D9/538E831F" Ref="#PWR024"  Part="1"
-AR Path="/538F26CD/538E831F" Ref="#PWR028"  Part="1"
-F 0 "#PWR028" H 8850 6950 30  0001 C CNN
+AR Path="/538C99D9/538E831F" Ref="#PWR023"  Part="1"
+AR Path="/538F26CD/538E831F" Ref="#PWR027"  Part="1"
+F 0 "#PWR023" H 8850 6950 30  0001 C CNN
 F 1 "GND" H 8850 6880 30  0001 C CNN
 F 2 "" H 8850 6950 60  0000 C CNN
@@
 $EndComp
 $Comp
-L GND #PWR025
+L GND #PWR024
 U 1 1 538E9F0A
 P 8050 6950
-AR Path="/538C99D9/538E9F0A" Ref="#PWR025"  Part="1"
-AR Path="/538F26CD/538E9F0A" Ref="#PWR029"  Part="1"
-F 0 "#PWR029" H 8050 6950 30  0001 C CNN
+AR Path="/538C99D9/538E9F0A" Ref="#PWR024"  Part="1"
+AR Path="/538F26CD/538E9F0A" Ref="#PWR028"  Part="1"
+F 0 "#PWR024" H 8050 6950 30  0001 C CNN
 F 1 "GND" H 8050 6880 30  0001 C CNN
 F 2 "" H 8050 6950 60  0000 C CNN
@@
 	7150 3700 7250 3800
 $Comp
-L GND #PWR026
+L GND #PWR025
 U 1 1 538F4EDD
 P 8850 4450
-AR Path="/538C99D9/538F4EDD" Ref="#PWR026"  Part="1"
-AR Path="/538F26CD/538F4EDD" Ref="#PWR030"  Part="1"
-F 0 "#PWR030" H 8850 4450 30  0001 C CNN
+AR Path="/538C99D9/538F4EDD" Ref="#PWR025"  Part="1"
+AR Path="/538F26CD/538F4EDD" Ref="#PWR029"  Part="1"
+F 0 "#PWR025" H 8850 4450 30  0001 C CNN
 F 1 "GND" H 8850 4380 30  0001 C CNN
 F 2 "" H 8850 4450 60  0000 C CNN
@@
 $EndComp
 $Comp
-L GND #PWR027
+L GND #PWR026
 U 1 1 538F4EDE
 P 8050 4450
-AR Path="/538C99D9/538F4EDE" Ref="#PWR027"  Part="1"
-AR Path="/538F26CD/538F4EDE" Ref="#PWR031"  Part="1"
-F 0 "#PWR031" H 8050 4450 30  0001 C CNN
+AR Path="/538C99D9/538F4EDE" Ref="#PWR026"  Part="1"
+AR Path="/538F26CD/538F4EDE" Ref="#PWR030"  Part="1"
+F 0 "#PWR026" H 8050 4450 30  0001 C CNN
 F 1 "GND" H 8050 4380 30  0001 C CNN
 F 2 "" H 8050 4450 60  0000 C CNN
@@
 Connection ~ 8850 4000
 $Comp
-L CONN\HDR\2MM\2R15\SHD J15
+L CONN\HDR\2MM\2R15\SHD J8
 U 1 1 53977A3A
 P 8450 3600
-AR Path="/538C99D9/53977A3A" Ref="J15"  Part="1"
-AR Path="/538F26CD/53977A3A" Ref="J17"  Part="1"
-F 0 "J17" H 8100 4450 60  0000 C CNN
+AR Path="/538C99D9/53977A3A" Ref="J8"  Part="1"
+AR Path="/538F26CD/53977A3A" Ref="J10"  Part="1"
+F 0 "J8" H 8100 4450 60  0000 C CNN
 F 1 "CONN\\HDR\\2MM\\2R15\\SHD" H 8450 4750 60  0001 C CNN
 F 2 "CONN_HDR_2MM_2R15_SHD" H 8450 4550 60  0000 C CNN
@@
 $EndComp
 $Comp
-L CONN\HDR\2MM\2R15\SHD J16
+L CONN\HDR\2MM\2R15\SHD J9
 U 1 1 53977A5C
 P 8450 6050
-AR Path="/538C99D9/53977A5C" Ref="J16"  Part="1"
-AR Path="/538F26CD/53977A5C" Ref="J18"  Part="1"
-F 0 "J18" H 8100 6900 60  0000 C CNN
+AR Path="/538C99D9/53977A5C" Ref="J9"  Part="1"
+AR Path="/538F26CD/53977A5C" Ref="J11"  Part="1"
+F 0 "J9" H 8100 6900 60  0000 C CNN
 F 1 "CONN\\HDR\\2MM\\2R15\\SHD" H 8450 7200 60  0001 C CNN
 F 2 "CONN_HDR_2MM_2R15_SHD" H 8450 7000 60  0000 C CNN

Commit message: Porcupine Version 2.
Changed lines of the file:
@@
 LIBS:valves
 LIBS:porcupine-cache
-EELAYER 24 0
+EELAYER 25 0
 EELAYER END
 $Descr B 17000 11000
 encoding utf-8
-Sheet 9 10
-Title "Parallella Breakout Daughtercard"
-Date "19 Jun 2014"
-Rev "*"
+Sheet 9 11
+Title "Parallella Breakout Daughtercard, Ver. 2"
+Date "17 feb 2015"
+Rev "A"
 Comp "Adapteva, Inc., 1666 Massachusetts Ave., Lexington, MA, 02420"
-Comment1 "Elink Connectors"
+Comment1 "Porcupine Top Level"
 Comment2 ""
 Comment3 ""
@@
 TXO_DATA_N[0..7]
 $Comp
-L GND #PWR023
+L GND #PWR017
 U 1 1 538E831F
 P 8850 6950
-AR Path="/538C99D9/538E831F" Ref="#PWR023"  Part="1"
-AR Path="/538F26CD/538E831F" Ref="#PWR027"  Part="1"
-F 0 "#PWR023" H 8850 6950 30  0001 C CNN
+AR Path="/538C99D9/538E831F" Ref="#PWR017"  Part="1"
+AR Path="/538F26CD/538E831F" Ref="#PWR021"  Part="1"
+F 0 "#PWR021" H 8850 6950 30  0001 C CNN
 F 1 "GND" H 8850 6880 30  0001 C CNN
 F 2 "" H 8850 6950 60  0000 C CNN
@@
 $EndComp
 $Comp
-L GND #PWR024
+L GND #PWR018
 U 1 1 538E9F0A
 P 8050 6950
-AR Path="/538C99D9/538E9F0A" Ref="#PWR024"  Part="1"
-AR Path="/538F26CD/538E9F0A" Ref="#PWR028"  Part="1"
-F 0 "#PWR024" H 8050 6950 30  0001 C CNN
+AR Path="/538C99D9/538E9F0A" Ref="#PWR018"  Part="1"
+AR Path="/538F26CD/538E9F0A" Ref="#PWR022"  Part="1"
+F 0 "#PWR022" H 8050 6950 30  0001 C CNN
 F 1 "GND" H 8050 6880 30  0001 C CNN
 F 2 "" H 8050 6950 60  0000 C CNN
@@
 	7150 3700 7250 3800
 $Comp
-L GND #PWR025
+L GND #PWR019
 U 1 1 538F4EDD
 P 8850 4450
-AR Path="/538C99D9/538F4EDD" Ref="#PWR025"  Part="1"
-AR Path="/538F26CD/538F4EDD" Ref="#PWR029"  Part="1"
-F 0 "#PWR025" H 8850 4450 30  0001 C CNN
+AR Path="/538C99D9/538F4EDD" Ref="#PWR019"  Part="1"
+AR Path="/538F26CD/538F4EDD" Ref="#PWR023"  Part="1"
+F 0 "#PWR023" H 8850 4450 30  0001 C CNN
 F 1 "GND" H 8850 4380 30  0001 C CNN
 F 2 "" H 8850 4450 60  0000 C CNN
@@
 $EndComp
 $Comp
-L GND #PWR026
+L GND #PWR020
 U 1 1 538F4EDE
 P 8050 4450
-AR Path="/538C99D9/538F4EDE" Ref="#PWR026"  Part="1"
-AR Path="/538F26CD/538F4EDE" Ref="#PWR030"  Part="1"
-F 0 "#PWR026" H 8050 4450 30  0001 C CNN
+AR Path="/538C99D9/538F4EDE" Ref="#PWR020"  Part="1"
+AR Path="/538F26CD/538F4EDE" Ref="#PWR024"  Part="1"
+F 0 "#PWR024" H 8050 4450 30  0001 C CNN
 F 1 "GND" H 8050 4380 30  0001 C CNN
 F 2 "" H 8050 4450 60  0000 C CNN
@@
 AR Path="/538C99D9/53977A3A" Ref="J8"  Part="1"
 AR Path="/538F26CD/53977A3A" Ref="J10"  Part="1"
-F 0 "J8" H 8100 4450 60  0000 C CNN
+F 0 "J10" H 8100 4450 60  0000 C CNN
 F 1 "CONN\\HDR\\2MM\\2R15\\SHD" H 8450 4750 60  0001 C CNN
 F 2 "CONN_HDR_2MM_2R15_SHD" H 8450 4550 60  0000 C CNN
@@
 AR Path="/538C99D9/53977A5C" Ref="J9"  Part="1"
 AR Path="/538F26CD/53977A5C" Ref="J11"  Part="1"
-F 0 "J9" H 8100 6900 60  0000 C CNN
+F 0 "J11" H 8100 6900 60  0000 C CNN
 F 1 "CONN\\HDR\\2MM\\2R15\\SHD" H 8450 7200 60  0001 C CNN
 F 2 "CONN_HDR_2MM_2R15_SHD" H 8450 7000 60  0000 C CNN
