File: boards/paracard-template/paracard-elink.sch (KiCad schematic (older format))
At the start: 1 part, among them P2 CONN\\SAMTEC\\BTH\\60

Commit message: Added E64 project with HDMI. Some cleanup to paracard template.
Connections:
- net GND: now also P2.11 (P11), P2.21 (P21), P2.31 (P31), P2.41 (P41), P2.51 (P51)
Changed lines of the file:
@@
 $Descr B 17000 11000
 encoding utf-8
-Sheet 5 6
+Sheet 3 6
 Title "Parallella Daughtercard"
 Date "09 May 2014"
@@
 	6800 3400 6900 3500
 Text HLabel 6300 2650 0    60   Input ~ 0
-RXI_DATA_N[7:0]
+RXI_DATA_N[0..7]
 Text HLabel 6300 2800 0    60   Input ~ 0
-RXI_DATA_P[7:0]
+RXI_DATA_P[0..7]
 Wire Bus Line
 	6950 5700 6950 6700
@@
 	10000 6200 10100 6300
 Text HLabel 10800 6700 2    60   Output ~ 0
-TXO_DATA_P[7:0]
-Text HLabel 10800 6850 2    60   Input ~ 0
-TXO_DATA_N[7:0]
+TXO_DATA_P[0..7]
+Text HLabel 10800 6850 2    60   Output ~ 0
+TXO_DATA_N[0..7]
 $Comp
 L GND #PWR03
@@
 AR Path="/5386858E/53875004" Ref="#PWR03"  Part="1"
 AR Path="/5387844C/53875004" Ref="#PWR07"  Part="1"
-F 0 "#PWR07" H 6500 7100 30  0001 C CNN
+F 0 "#PWR03" H 6500 7100 30  0001 C CNN
 F 1 "GND" H 6500 7030 30  0001 C CNN
 F 2 "" H 6500 7100 60  0000 C CNN
@@
 L GND #PWR04
 U 1 1 53875018
-P 10600 7100
+P 10400 7100
 AR Path="/5386858E/53875018" Ref="#PWR04"  Part="1"
 AR Path="/5387844C/53875018" Ref="#PWR08"  Part="1"
-F 0 "#PWR08" H 10600 7100 30  0001 C CNN
-F 1 "GND" H 10600 7030 30  0001 C CNN
-F 2 "" H 10600 7100 60  0000 C CNN
-F 3 "" H 10600 7100 60  0000 C CNN
-	1    10600 7100
+F 0 "#PWR04" H 10400 7100 30  0001 C CNN
+F 1 "GND" H 10400 7030 30  0001 C CNN
+F 2 "" H 10400 7100 60  0000 C CNN
+F 3 "" H 10400 7100 60  0000 C CNN
+	1    10400 7100
 	1    0    0    -1
 $EndComp
@@
 AR Path="/5386858E/53893761" Ref="P2"  Part="1"
 AR Path="/5387844C/53893761" Ref="P4"  Part="1"
-F 0 "P4" H 8450 6550 60  0000 C CNN
+F 0 "P2" H 8450 6550 60  0000 C CNN
 F 1 "CONN\\SAMTEC\\BTH\\60" V 8350 4850 60  0000 C CNN
 F 2 "CONN_SAMTEC_BTH_60" V 8550 4850 60  0001 C CNN

Commit message: Ready for full review.
Parts:
- P2: MFR Samtec -> (none); Manufacturer (none) -> Samtec
Changed lines of the file:
@@
 F 1 "CONN\\SAMTEC\\BTH\\60" V 8350 4850 60  0000 C CNN
 F 2 "CONN_SAMTEC_BTH_60" V 8550 4850 60  0001 C CNN
-F 3 "/mnt/windowsC/Adapteva/Fred-suppliers/Suppliers/www.samtec.com/BTH-XXX-XX-X-D-XX-MKT.pdf" H 8550 5750 60  0001 C CNN
+F 3 "" H 8550 5750 60  0001 C CNN
 F 4 "BTH-030-01-F-D-A" V 8450 4850 80  0000 C CNN "MFRPN"
-F 5 "Samtec" V 8450 3650 60  0000 C CNN "MFR"
+F 5 "Samtec" V 8450 3650 60  0000 C CNN "Manufacturer"
 	1    8450 4850
 	1    0    0    -1
