File: boards/paracard-template/paracard-gpio.sch (KiCad schematic (older format))
At the start: 1 part, among them P1 CONN\\SAMTEC\\BTH\\60

Commit message: Added E64 project with HDMI. Some cleanup to paracard template.
Connections:
- net VGPIO: now also P1.1 (P1)
Changed lines of the file:
@@
 GPIO_P23
 Text HLabel 8650 2850 0    60   BiDi ~ 0
-GPIO_N[23:0]
+GPIO_N[0..23]
 Text HLabel 8650 3000 0    60   BiDi ~ 0
-GPIO_P[23:0]
+GPIO_P[0..23]
 Text Label 5700 2800 2    60   ~ 0
 GPIO_N0
@@
 	6150 5300 6250 5200
 Text Label 6750 2700 2    60   ~ 0
-GPIO[47:0]
+GPIO[0..47]
 Text HLabel 6850 2700 2    60   BiDi ~ 0
-GPIO[47:0]
+GPIO[0..47]
 Entry Wire Line
 	6150 5100 6250 5000
@@
 	5200 2700 5300 2800
 Text Label 5900 2500 2    60   ~ 0
-GPIO_N[23:0]
+GPIO_N[0..23]
 Text Label 6100 8000 2    60   ~ 0
-GPIO_P[23:0]
+GPIO_P[0..23]
 Text Notes 6500 6900 1    80   ~ 0
 Aliases between differential and single-ended GPIOs
@@
 	9800 3700 9950 3700
 Wire Wire Line
-	11050 3700 11050 3300
+	11050 3300 11050 3700
 Wire Bus Line
 	9200 2850 9200 6400
@@
 	5200 8000 6150 8000
 Wire Wire Line
-	11250 3300 9650 3300
-Wire Wire Line
 	9800 3700 9800 3300
-Connection ~ 9800 3300
 Wire Wire Line
 	11950 4200 11950 6700
@@
 	1    0    0    -1
 $EndComp
+Wire Wire Line
+	9650 3300 11050 3300
+Connection ~ 9800 3300
 $EndSCHEMATC

Commit message: Ready for full review.
Parts:
- P1: MFR Samtec -> (none); Manufacturer (none) -> Samtec
Changed lines of the file:
@@
 F 1 "CONN\\SAMTEC\\BTH\\60" V 10350 5150 60  0000 C CNN
 F 2 "CONN_SAMTEC_BTH_60" V 10550 5150 60  0001 C CNN
-F 3 "/mnt/windowsC/Adapteva/Fred-suppliers/Suppliers/www.samtec.com/BTH-XXX-XX-X-D-XX-MKT.pdf" H 10550 6050 60  0001 C CNN
+F 3 "" H 10550 6050 60  0001 C CNN
 F 4 "BTH-030-01-F-D-A" V 10450 5150 80  0000 C CNN "MFRPN"
-F 5 "Samtec" V 10450 3950 60  0000 C CNN "MFR"
+F 5 "Samtec" V 10450 3950 60  0000 C CNN "Manufacturer"
 	1    10450 5150
 	1    0    0    -1
@@
 	9650 3300 11050 3300
 Connection ~ 9800 3300
+Text Label 9850 2850 0    60   ~ 0
+GPIO_N[0..23]
+Text Label 9850 3000 0    60   ~ 0
+GPIO_P[0..23]
 $EndSCHEMATC
