File: boards/paracard-template/paracard-power.sch (KiCad schematic (older format))
At the start: 1 part, among them P3 CONN\\SAMTEC\\BTH\\60

Commit message: Added E64 project with HDMI. Some cleanup to paracard template.
Connections:
- net labels added: DSP_XID[0..3], DSP_YID[0..3], REG_EN[1..4]
- net labels removed: DSP_XID[3:0], DSP_YID[3:0], REG_EN[4:1]
Changed lines of the file:
@@
 REG_EN3
 Text Label 6500 4650 2    60   ~ 0
-REG_EN[4:1]
+REG_EN[1..4]
 Text HLabel 5850 4650 0    60   Input ~ 0
-REG_EN[4:1]
+REG_EN[1..4]
 NoConn ~ 8650 4000
 Text HLabel 10550 4000 2    60   BiDi ~ 0
@@
 	5850 5050 6550 5050
 Text Label 5900 4850 0    60   ~ 0
-DSP_YID[3:0]
+DSP_YID[0..3]
 Text Label 5900 5050 0    60   ~ 0
-DSP_XID[3:0]
+DSP_XID[0..3]
 Text HLabel 5850 4850 0    60   Input ~ 0
-DSP_YID[3:0]
+DSP_YID[0..3]
 Text HLabel 5850 5050 0    60   Input ~ 0
-DSP_XID[3:0]
+DSP_XID[0..3]
 Text HLabel 7750 4700 0    60   Input ~ 0
 UART_RX

Commit message: Ready for full review.
Parts:
- P3: MFR Samtec -> (none); Manufacturer (none) -> Samtec
Connections:
- net labels added: SPARE
- wire segments 64 -> 65
- no-connect marks 1 -> 0
Changed lines of the file:
@@
 Text HLabel 5850 4650 0    60   Input ~ 0
 REG_EN[1..4]
-NoConn ~ 8650 4000
 Text HLabel 10550 4000 2    60   BiDi ~ 0
 PROG_IO
@@
 F 1 "CONN\\SAMTEC\\BTH\\60" V 9050 5050 60  0000 C CNN
 F 2 "CONN_SAMTEC_BTH_60" V 9250 5050 60  0001 C CNN
-F 3 "/mnt/windowsC/Adapteva/Fred-suppliers/Suppliers/www.samtec.com/BTH-XXX-XX-X-D-XX-MKT.pdf" H 9250 5950 60  0001 C CNN
+F 3 "" H 9250 5950 60  0001 C CNN
 F 4 "BTH-030-01-F-D-A" V 9150 5050 80  0000 C CNN "MFRPN"
-F 5 "Samtec" V 9150 3850 60  0000 C CNN "MFR"
+F 5 "Samtec" V 9150 3850 60  0000 C CNN "Manufacturer"
 	1    9150 5050
 	1    0    0    -1
 $EndComp
+Text HLabel 7750 4000 0    60   BiDi ~ 0
+SPARE
+Wire Wire Line
+	7750 4000 8650 4000
 $EndSCHEMATC
